File: 14_Demi_Pont_H_99.kicad_pcb (KiCad board)
At the start: 2 copper layers, 20.3 x 20.3 mm, 17 parts, among them J1 Conn_01x01, J2 Conn_01x01, J3 Conn_01x01, J4 Conn_01x01, J5 Conn_01x01, J6 Conn_01x01, J7 Conn_01x01, Q1 FDS8884, Q2 FDS8884, U1 IMP3201

Commit message: maj split libraires
Parts:
- J1, J2, J3, J4, J5, J6, J7: footprint Chimere:Castellated_conn -> Chimere_mods:Castellated_conn
