File: 14_Demi_Pont_H_99.sch (KiCad schematic (older format))
At the start: 17 parts, among them J1 Conn_01x01, J2 Conn_01x01, J3 Conn_01x01, J4 Conn_01x01, J5 Conn_01x01, J6 Conn_01x01, J7 Conn_01x01, Q1 FDS8884, Q2 FDS8884, U1 IMP3201

Commit message: maj split libraires
Parts:
- J1, J2, J3, J4, J5, J6, J7: footprint Chimere:Castellated_conn -> Chimere_mods:Castellated_conn
- Q1, Q2: symbol Chimere:FDS6630A -> Chimere_comps:FDS6630A
- U1: symbol Chimere:IMP3201 -> Chimere_comps:IMP3201
Changed lines of the file:
@@
 F 0 "J5" H 7230 3942 50  0000 L CNN
 F 1 "Conn_01x01" H 7230 3851 50  0000 L CNN
-F 2 "Chimere:Castellated_conn" H 7150 3900 50  0001 C CNN
+F 2 "Chimere_mods:Castellated_conn" H 7150 3900 50  0001 C CNN
 F 3 "~" H 7150 3900 50  0001 C CNN
 	1    7150 3900
@@
 F 0 "J6" H 7230 4142 50  0000 L CNN
 F 1 "Conn_01x01" H 7230 4051 50  0000 L CNN
-F 2 "Chimere:Castellated_conn" H 7150 4100 50  0001 C CNN
+F 2 "Chimere_mods:Castellated_conn" H 7150 4100 50  0001 C CNN
 F 3 "~" H 7150 4100 50  0001 C CNN
 	1    7150 4100
@@
 F 0 "J4" H 7230 3742 50  0000 L CNN
 F 1 "Conn_01x01" H 7230 3651 50  0000 L CNN
-F 2 "Chimere:Castellated_conn" H 7150 3700 50  0001 C CNN
+F 2 "Chimere_mods:Castellated_conn" H 7150 3700 50  0001 C CNN
 F 3 "~" H 7150 3700 50  0001 C CNN
 	1    7150 3700
@@
 F 0 "J1" H 7230 3192 50  0000 L CNN
 F 1 "Conn_01x01" H 7230 3101 50  0000 L CNN
-F 2 "Chimere:Castellated_conn" H 7150 3150 50  0001 C CNN
+F 2 "Chimere_mods:Castellated_conn" H 7150 3150 50  0001 C CNN
 F 3 "~" H 7150 3150 50  0001 C CNN
 	1    7150 3150
@@
 F 0 "J3" H 7230 3567 50  0000 L CNN
 F 1 "Conn_01x01" H 7230 3476 50  0000 L CNN
-F 2 "Chimere:Castellated_conn" H 7150 3525 50  0001 C CNN
+F 2 "Chimere_mods:Castellated_conn" H 7150 3525 50  0001 C CNN
 F 3 "~" H 7150 3525 50  0001 C CNN
 	1    7150 3525
@@
 GND
 $Comp
-L Chimere:FDS6630A Q2
+L Chimere_comps:FDS6630A Q2
 U 1 1 6078CBA9
 P 5100 4425
@@
 	4150 3700 4250 3700
 $Comp
-L Chimere:FDS6630A Q1
+L Chimere_comps:FDS6630A Q1
 U 1 1 60B53179
 P 5100 3700
@@
 imp3201\nC72885
 $Comp
-L Chimere:IMP3201 U1
+L Chimere_comps:IMP3201 U1
 U 1 1 60B5A254
 P 3050 3925
@@
 F 0 "J2" H 7230 3367 50  0000 L CNN
 F 1 "Conn_01x01" H 7230 3276 50  0000 L CNN
-F 2 "Chimere:Castellated_conn" H 7150 3325 50  0001 C CNN
+F 2 "Chimere_mods:Castellated_conn" H 7150 3325 50  0001 C CNN
 F 3 "~" H 7150 3325 50  0001 C CNN
 	1    7150 3325
@@
 F 0 "J7" H 7230 4342 50  0000 L CNN
 F 1 "Conn_01x01" H 7230 4251 50  0000 L CNN
-F 2 "Chimere:Castellated_conn" H 7150 4300 50  0001 C CNN
+F 2 "Chimere_mods:Castellated_conn" H 7150 4300 50  0001 C CNN
 F 3 "~" H 7150 4300 50  0001 C CNN
 	1    7150 4300
